Commit message: camera fixed

File: CODE/Enviornment/xml_models/base-camera-stand/robot.urdf (robot description, URDF)
Before this commit: robot base-camera-stand, 3 links, 2 joints
Joints:
- joint base-and-bottom-plate: origin xyz=0.00286592 -0.0153152 -0.0180122 rpy=1.2557e-08 1.1562e-08 1.26e-10 -> xyz=0 0 0.02 rpy=-0 0 -0
- joint base-and-camera-stand: origin xyz=0.165366 0.00468478 0.0169878 rpy=1.5708 1.1562e-08 1.26e-10 -> xyz=0.1625 0.02 0.055 rpy=1.5708 0 -0
